File: Shield/v1.0/Trimble Thunderbolt Monitor Shield v1.0.brd (EAGLE design)
At the start: 60.9 x 54.3 mm, 31 parts, among them Q1 2N2222, U2 MAX232PTH

Commit message: Fixed some silkscreen issues
Other:
- board text added: "(3) (2) (5)"
- board text removed: "(2) (3) (5)"
Changed lines of the file:
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@@
 <?xml version="1.0" encoding="utf-8"?>
 <!DOCTYPE eagle SYSTEM "eagle.dtd">
-<eagle version="6.4">
+<eagle version="6.5.0">
 <drawing>
 <settings>
@@
 3) Minor Alarm
 4) Major Alarm</text>
-<text x="79.375" y="55.88" size="0.762" layer="21" font="vector" rot="R180">(2) (3) (5)</text>
+<text x="79.375" y="55.88" size="0.762" layer="21" font="vector" rot="R180">(3) (2) (5)</text>
 </plain>
 <attributes>

Commit message: Fixed some ERC issues
Parts:
- S1: value RIGHT -> (none)
- S2: value UP -> (none)
- S3: value DOWN -> (none)
- S4: value LEFT -> (none)
- S5: value SELECT -> (none)
Changed lines of the file:
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@@
 <element name="JP1" library="pinhead" package="1X16" value="HD44780" x="45.72" y="83.82"/>
 <element name="U2" library="SparkFun" package="DIL16" value="MAX232PTH" x="74.93" y="68.58" rot="R270"/>
-<element name="S2" library="SparkFun" package="TACTILE-PTH" value="UP" x="29.21" y="52.07" smashed="yes">
+<element name="S2" library="SparkFun" package="TACTILE-PTH" value="" x="29.21" y="52.07" smashed="yes">
 <attribute name="NAME" x="32.385" y="51.435" size="1.27" layer="25" ratio="10"/>
 </element>
-<element name="S3" library="SparkFun" package="TACTILE-PTH" value="DOWN" x="29.21" y="44.45" smashed="yes">
+<element name="S3" library="SparkFun" package="TACTILE-PTH" value="" x="29.21" y="44.45" smashed="yes">
 <attribute name="NAME" x="32.385" y="43.815" size="1.27" layer="25" ratio="10"/>
 </element>
-<element name="S4" library="SparkFun" package="TACTILE-PTH" value="LEFT" x="39.37" y="52.07" smashed="yes">
+<element name="S4" library="SparkFun" package="TACTILE-PTH" value="" x="39.37" y="52.07" smashed="yes">
 <attribute name="NAME" x="42.545" y="51.435" size="1.27" layer="25" ratio="10"/>
 </element>
-<element name="S5" library="SparkFun" package="TACTILE-PTH" value="SELECT" x="58.42" y="52.07" smashed="yes">
+<element name="S5" library="SparkFun" package="TACTILE-PTH" value="" x="58.42" y="52.07" smashed="yes">
 <attribute name="NAME" x="61.595" y="51.435" size="1.27" layer="25" ratio="10"/>
 </element>
@@
 <element name="C3" library="SparkFun" package="CPOL-RADIAL-10UF-25V" value="1uF" x="74.93" y="82.55" rot="R180"/>
 <element name="C4" library="SparkFun" package="CPOL-RADIAL-10UF-25V" value="1uF" x="66.04" y="62.23" rot="R270"/>
-<element name="S1" library="SparkFun" package="TACTILE-PTH" value="RIGHT" x="49.53" y="52.07" smashed="yes">
+<element name="S1" library="SparkFun" package="TACTILE-PTH" value="" x="49.53" y="52.07" smashed="yes">
 <attribute name="NAME" x="52.705" y="51.435" size="1.27" layer="25" ratio="10"/>
 </element>
